File: RGBModule/RGBModule.sch (KiCad schematic (older format))
At the start: 5 parts

Commit message: Netlist y footprints asociados
Parts:
- LED1: renamed from LED?; footprint RGBLED5050 -> SparkFun-LED:LED-TRICOLOR-5050
- P1: renamed from P?; footprint (none) -> Connectors_JST:JST_PH_S4B-PH-K_04x2.00mm_Angled
- R1, R2, R3: renamed from R?; footprint (none) -> Resistors_SMD:R_0805
Changed lines of the file:
@@
 $EndDescr
 $Comp
-L RGBLED5050 LED?
+L RGBLED5050 LED1
 U 1 1 592305F2
 P 5550 3500
-F 0 "LED?" H 5400 3850 50  0000 L BNN
+F 0 "LED1" H 5400 3850 50  0000 L BNN
 F 1 "RGBLED5050" H 5550 3500 50  0001 L BNN
-F 2 "RGBLED5050" H 5580 3650 20  0001 C CNN
+F 2 "SparkFun-LED:LED-TRICOLOR-5050" H 5580 3650 20  0001 C CNN
 F 3 "" H 5550 3500 60  0001 C CNN
 	1    5550 3500
@@
 $EndComp
 $Comp
-L R R?
+L R R1
 U 1 1 59230805
 P 5000 3300
-F 0 "R?" V 5080 3300 50  0000 C CNN
+F 0 "R1" V 5080 3300 50  0000 C CNN
 F 1 "330" V 5000 3300 50  0000 C CNN
-F 2 "" V 4930 3300 50  0001 C CNN
+F 2 "Resistors_SMD:R_0805" V 4930 3300 50  0001 C CNN
 F 3 "" H 5000 3300 50  0001 C CNN
 	1    5000 3300
@@
 $EndComp
 $Comp
-L R R?
+L R R2
 U 1 1 59230856
 P 5000 3500
-F 0 "R?" V 5080 3500 50  0000 C CNN
+F 0 "R2" V 5080 3500 50  0000 C CNN
 F 1 "330" V 5000 3500 50  0000 C CNN
-F 2 "" V 4930 3500 50  0001 C CNN
+F 2 "Resistors_SMD:R_0805" V 4930 3500 50  0001 C CNN
 F 3 "" H 5000 3500 50  0001 C CNN
 	1    5000 3500
@@
 $EndComp
 $Comp
-L R R?
+L R R3
 U 1 1 59230874
 P 5000 3700
-F 0 "R?" V 5080 3700 50  0000 C CNN
+F 0 "R3" V 5080 3700 50  0000 C CNN
 F 1 "470" V 5000 3700 50  0000 C CNN
-F 2 "" V 4930 3700 50  0001 C CNN
+F 2 "Resistors_SMD:R_0805" V 4930 3700 50  0001 C CNN
 F 3 "" H 5000 3700 50  0001 C CNN
 	1    5000 3700
@@
 Wire Wire Line
 	5150 3700 5350 3700
-$Comp
-L GND #PWR?
-U 1 1 59230922
-P 5950 3850
-F 0 "#PWR?" H 5950 3600 50  0001 C CNN
-F 1 "GND" H 5950 3700 50  0000 C CNN
-F 2 "" H 5950 3850 50  0001 C CNN
-F 3 "" H 5950 3850 50  0001 C CNN
-	1    5950 3850
-	1    0    0    -1
-$EndComp
 Wire Wire Line
 	5750 3700 5950 3700
 Wire Wire Line
 	5950 3300 5950 3850
-Wire Wire Line
-	5750 3500 5950 3500
 Connection ~ 5950 3700
 Wire Wire Line
@@
 BLUE
 $Comp
-L CONN_01X04 P?
+L CONN_01X04 P1
 U 1 1 59230A2F
 P 3900 4650
-F 0 "P?" H 3900 4900 50  0000 C CNN
+F 0 "P1" H 3900 4900 50  0000 C CNN
 F 1 "CONN_01X04" V 4000 4650 50  0000 C CNN
-F 2 "" H 3900 4650 50  0001 C CNN
+F 2 "Connectors_JST:JST_PH_S4B-PH-K_04x2.00mm_Angled" H 3900 4650 50  0001 C CNN
 F 3 "" H 3900 4650 50  0001 C CNN
 	1    3900 4650
 	-1   0    0    1
-$EndComp
-$Comp
-L GND #PWR?
-U 1 1 59230E0E
-P 4150 4950
-F 0 "#PWR?" H 4150 4700 50  0001 C CNN
-F 1 "GND" H 4150 4800 50  0000 C CNN
-F 2 "" H 4150 4950 50  0001 C CNN
-F 3 "" H 4150 4950 50  0001 C CNN
-	1    4150 4950
-	1    0    0    -1
 $EndComp
 Wire Wire Line
@@
 Text GLabel 4250 4700 2    39   Input ~ 0
 RED
+$Comp
+L PWR_FLAG #FLG01
+U 1 1 59231234
+P 6600 7350
+F 0 "#FLG01" H 6600 7425 50  0001 C CNN
+F 1 "PWR_FLAG" H 6600 7500 50  0000 C CNN
+F 2 "" H 6600 7350 50  0001 C CNN
+F 3 "" H 6600 7350 50  0001 C CNN
+	1    6600 7350
+	1    0    0    -1
+$EndComp
+$Comp
+L GND #PWR02
+U 1 1 592315AB
+P 5950 3850
+F 0 "#PWR02" H 5950 3600 50  0001 C CNN
+F 1 "GND" H 5950 3700 50  0000 C CNN
+F 2 "" H 5950 3850 50  0001 C CNN
+F 3 "" H 5950 3850 50  0001 C CNN
+	1    5950 3850
+	1    0    0    -1
+$EndComp
+$Comp
+L GND #PWR03
+U 1 1 59231608
+P 4150 4950
+F 0 "#PWR03" H 4150 4700 50  0001 C CNN
+F 1 "GND" H 4150 4800 50  0000 C CNN
+F 2 "" H 4150 4950 50  0001 C CNN
+F 3 "" H 4150 4950 50  0001 C CNN
+	1    4150 4950
+	1    0    0    -1
+$EndComp
+$Comp
+L GND #PWR04
+U 1 1 5923165E
+P 6600 7450
+F 0 "#PWR04" H 6600 7200 50  0001 C CNN
+F 1 "GND" H 6600 7300 50  0000 C CNN
+F 2 "" H 6600 7450 50  0001 C CNN
+F 3 "" H 6600 7450 50  0001 C CNN
+	1    6600 7450
+	1    0    0    -1
+$EndComp
+Wire Wire Line
+	6600 7350 6600 7450
+Wire Wire Line
+	5950 3500 5750 3500
 $EndSCHEMATC

Commit message: Logo y conector cambiado
Parts:
- P1: footprint Connectors_JST:JST_PH_S4B-PH-K_04x2.00mm_Angled -> Pin_Headers:Pin_Header_Angled_1x04_Pitch2.54mm
Changed lines of the file:
@@
 EESchema Schematic File Version 2
-LIBS:power
-LIBS:device
-LIBS:transistors
-LIBS:conn
-LIBS:linear
-LIBS:regul
+LIBS:74xgxx
 LIBS:74xx
-LIBS:cmos4000
-LIBS:adc-dac
-LIBS:memory
-LIBS:xilinx
-LIBS:microcontrollers
-LIBS:dsp
-LIBS:microchip
-LIBS:analog_switches
-LIBS:motorola
-LIBS:texas
-LIBS:intel
-LIBS:audio
-LIBS:interface
-LIBS:digital-audio
-LIBS:philips
-LIBS:display
-LIBS:cypress
-LIBS:siliconi
-LIBS:opto
-LIBS:atmel
-LIBS:contrib
-LIBS:valves
-LIBS:74xgxx
 LIBS:5050_ws2811
 LIBS:a4988-module
@@
 LIBS:actel
 LIBS:adafruit
+LIBS:adc-dac
 LIBS:adxl345
 LIBS:allegro
@@
 LIBS:AMS1117
 LIBS:analog_devices
+LIBS:analog_switches
 LIBS:ant
 LIBS:at24c64
+LIBS:atmel
+LIBS:audio
 LIBS:battery_management
 LIBS:bbd
@@
 LIBS:bosch
 LIBS:brooktre
+LIBS:cmos4000
 LIBS:cmos_ieee
+LIBS:conn
+LIBS:contrib
 LIBS:cp2103
 LIBS:CP2102
+LIBS:cypress
 LIBS:dc-dc
+LIBS:device
 LIBS:dht11
+LIBS:digital-audio
 LIBS:diode
+LIBS:display
+LIBS:dsp
 LIBS:elec-unifil
 LIBS:er-oled-ssd1306
@@
 LIBS:HC164
 LIBS:hlk-rm04
+LIBS:intel
+LIBS:interface
 LIBS:ir
 LIBS:irf7907
@@
 LIBS:Lattice
 LIBS:LilyPad-Wearables
+LIBS:linear
 LIBS:LM2575
 LIBS:logo
@@
 LIBS:MCP3208
 LIBS:mechanical
+LIBS:memory
+LIBS:microchip
 LIBS:microchip_dspic33dsc
 LIBS:microchip_pic10mcu
@@
 LIBS:microchip_pic18mcu
 LIBS:microchip_pic32mcu
+LIBS:microcontrollers
 LIBS:miniusb
 LIBS:motor_drivers
+LIBS:motorola
 LIBS:motors
 LIBS:mp2109dq
@@
 LIBS:OF5032
 LIBS:onsemi
+LIBS:opto
 LIBS:Oscillators
+LIBS:philips
 LIBS:pl2303
 LIBS:pogopin
+LIBS:power
 LIBS:powerint
 LIBS:powerjack
@@
 LIBS:pt4115
 LIBS:references
+LIBS:regul
 LIBS:relays
 LIBS:rfcom
@@
 LIBS:sensors
 LIBS:silabs
+LIBS:siliconi
 LIBS:smd oscillator
 LIBS:songle_relay
@@
 LIBS:Teensy_3_and_LC_Series_Boards_v1.1
 LIBS:test
+LIBS:texas
 LIBS:texas-msp
 LIBS:tlv70233
 LIBS:tp4056
 LIBS:transf
+LIBS:transistors
 LIBS:ts812c
 LIBS:ttl_ieee
@@
 LIBS:usb_ax2
 LIBS:User-Submitted
+LIBS:valves
 LIBS:video
 LIBS:w25q32bv
@@
 LIBS:XC9572-TQ100
 LIBS:Xicor
+LIBS:xilinx
 LIBS:xilinx_spartan3_virtex4_and_5
 LIBS:zetex
@@
 LIBS:рэс-49
 LIBS:тпг-1
+LIBS:RGBModule-cache
 EELAYER 25 0
 EELAYER END
@@
 F 0 "P1" H 3900 4900 50  0000 C CNN
 F 1 "CONN_01X04" V 4000 4650 50  0000 C CNN
-F 2 "Connectors_JST:JST_PH_S4B-PH-K_04x2.00mm_Angled" H 3900 4650 50  0001 C CNN
+F 2 "Pin_Headers:Pin_Header_Angled_1x04_Pitch2.54mm" H 3900 4650 50  0001 C CNN
 F 3 "" H 3900 4650 50  0001 C CNN
 	1    3900 4650
